File: Lamp Logic Board/Lamp Logic Board_2.brd (EAGLE design)
At the start: 41.5 x 83.4 mm, 45 parts, among them U1 ESP32-WROVER-IB, U2 SN74HCT245DWR, U4 LM50, U5 SPIOLED_STANDOFF, U6 MSGEQ7DIL

Commit message: hahaha
Connections:
- removed net N$16: U1.37
- removed net VDD3V3_TEMP-OUT: U1.14
- net LEDS8_3V3: now also U1.37; no longer U1.36
- net MSGEQ_RST: now also U1.4
- net OUTA: now also U1.17; no longer U1.11
- net OUTB: now also U1.18; no longer U1.12
- net ROTARY_BUTTON_IN: now also U1.13; no longer U1.4
- net VDD3V3_TEMP_OUT: now also U1.14
Routing:
- net VDD3V3_TEMP_OUT: track 0.00 -> 15.4 mm
- net MSGEQ_RST: track 0.00 -> 13.2 mm, vias 0 -> 1
- net ROTARY_BUTTON_IN: track 57.7 -> 48.2 mm
- net OUTB: track 41.8 -> 37.2 mm
- net GND: track 89.2 -> 84.7 mm
- net OUTA: track 43.8 -> 39.4 mm
- net LEDS8_3V3: track 51.3 -> 52.1 mm
- net LEDSDIAG_3V3: track 23.6 -> 22.9 mm

Commit message: omg
Parts:
- moved U$3 2.95 mm to (35.8, 63.8)
- moved MICROSD_CONN 1.45 mm to (32.5, 53.7)
- moved U1 1.35 mm to (25.1, 78.1)
- moved C4 1.28 mm to (9.82, 68.2), turned to 0 degrees
- moved R2 1.22 mm to (20.1, 24.1)
- moved R14 1.18 mm to (16.9, 30.5)
- moved R3 1.06 mm to (22.8, 24.1)
- moved R13 1.03 mm to (16.3, 24.1)
- moved R4 0.92 mm to (25.5, 24.2)
- moved R5 0.78 mm to (28.2, 24.1)
- moved R6 0.66 mm to (30.9, 24.1)
- moved R7 0.55 mm to (33.6, 24.1)
- moved R8 0.48 mm to (36.3, 24.1)
- moved R9 0.45 mm to (39.0, 24.1)
- moved C6 0.20 mm to (13.0, 46.0)
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Connections:
- net LEDS8_3V3: now also U1.36; no longer U1.37
- net MSGEQ_RST: now also U1.12; no longer U1.4
Routing:
- net MSGEQ_RST: track 13.2 -> 25.6 mm, vias 1 -> 2
- net GND: track 84.7 -> 97.0 mm
- net SCK: track 47.4 -> 52.7 mm
- net IO0: track 70.3 -> 73.9 mm
- net SD_D1: track 18.2 -> 20.4 mm
- net VDD3V3: track 150.6 -> 152.7 mm
- net SD_D0: track 18.6 -> 20.6 mm
- net N$14: track 8.25 -> 10.0 mm
- net SD_SCK: track 18.2 -> 19.9 mm
- net OUTB: track 37.2 -> 35.5 mm
- net MOSI: track 42.6 -> 44.2 mm
- net N$13: track 6.13 -> 7.74 mm
- net VDD3V3_TEMP_OUT: track 15.4 -> 16.9 mm
- net MISO: track 38.2 -> 39.6 mm
- net LEDS3_3V3: track 37.6 -> 39.0 mm
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Other:
- board size 41.5 x 83.4 mm -> 41.5 x 84.8 mm

Commit message: Another day closer to death...
Parts:
- moved C3 0.53 mm to (19.6, 50.0)
- moved U$4 0.51 mm to (17.3, 15.1)
- moved R13 0.51 mm to (16.2, 23.6)
- moved R15 0.43 mm to (13.8, 13.1)
- moved U2 0.43 mm to (33.3, 34.3)
- moved R2 0.40 mm to (20.1, 23.7)
- moved R3 0.40 mm to (22.8, 23.8)
- moved R4 0.40 mm to (25.5, 23.8)
- moved R5 0.40 mm to (28.2, 23.8)
- moved R6 0.40 mm to (30.9, 23.8)
- moved R7 0.40 mm to (33.6, 23.8)
- moved R8 0.40 mm to (36.3, 23.8)
- moved R9 0.40 mm to (39.0, 23.8)
- moved R1 0.35 mm to (23.5, 38.9)
- moved C7 0.18 mm to (39.2, 12.4)
Connections:
- net GAIN: now also U1.11
Routing:
- net GAIN: track 0.00 -> 22.3 mm, vias 0 -> 1
- net SD_CS: track 47.1 -> 28.9 mm, vias 2 -> 4
- net ROTARY_BUTTON_IN: track 47.7 -> 50.2 mm
- net N$7: track 7.16 -> 9.31 mm
- net IO0: track 73.9 -> 72.3 mm
- net N$3: track 12.3 -> 13.1 mm
- net MISO: track 39.6 -> 40.2 mm
- net LEDS1_5V: track 12.5 -> 11.9 mm
- net LEDS7_5V: track 13.0 -> 12.3 mm
- net LEDS4_5V: track 12.8 -> 12.2 mm
- net N$14: track 10.0 -> 9.51 mm
- net LEDS8_5V: track 13.0 -> 12.5 mm
- net LEDS6_5V: track 12.8 -> 12.3 mm
- net LEDS3_5V: track 12.6 -> 12.1 mm
