File: Lamp Logic Board/Lamp Logic Board_2.sch (EAGLE design)
At the start: 45 parts, among them U1 ESP32-WROVER-IB, U2 SN74HCT245DWR, U3 LM1117MP-1.8, U4 LM50, U5 SPIOLED_STANDOFF, U6 MSGEQ7DIL

Commit message: hahaha
Connections:
- removed net N$16: U1.IO23
- removed net VDD3V3_TEMP-OUT: U1.IO12
- net LEDS8_3V3: now also U1.IO23; no longer U1.IO22
- net MSGEQ_RST: now also U1.SENSOR_VP
- net OUTA: now also U1.SHD/SD2; no longer U1.IO26
- net OUTB: now also U1.SWP/SD3; no longer U1.IO27
- net ROTARY_BUTTON_IN: now also U1.IO14; no longer U1.SENSOR_VP
- net VDD3V3_TEMP_OUT: now also U1.IO12
Other:
- moved on the sheet: R1
Changed lines of the file:
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@@
 <attribute name="VALUE" x="377.19" y="171.958" size="1.778" layer="96"/>
 </instance>
-<instance part="R1" gate="G$1" x="220.98" y="114.3" smashed="yes">
-<attribute name="NAME" x="214.63" y="113.2586" size="1.778" layer="95"/>
-<attribute name="VALUE" x="219.71" y="116.078" size="1.778" layer="96"/>
+<instance part="R1" gate="G$1" x="243.84" y="111.76" smashed="yes">
+<attribute name="NAME" x="237.49" y="110.7186" size="1.778" layer="95"/>
+<attribute name="VALUE" x="242.57" y="113.538" size="1.778" layer="96"/>
 </instance>
 <instance part="R10" gate="G$1" x="99.06" y="132.08" smashed="yes">
@@
 <segment>
 <pinref part="U1" gate="G$1" pin="RXD0"/>
-<wire x1="210.82" y1="116.84" x2="218.44" y2="116.84" width="0.1524" layer="91"/>
-<wire x1="218.44" y1="116.84" x2="218.44" y2="119.38" width="0.1524" layer="91"/>
-<wire x1="218.44" y1="119.38" x2="226.06" y2="119.38" width="0.1524" layer="91"/>
-<wire x1="226.06" y1="119.38" x2="226.06" y2="116.84" width="0.1524" layer="91"/>
-<wire x1="226.06" y1="116.84" x2="233.68" y2="116.84" width="0.1524" layer="91"/>
+<wire x1="210.82" y1="116.84" x2="233.68" y2="114.3" width="0.1524" layer="91"/>
 <label x="228.6" y="116.84" size="1.778" layer="95"/>
 </segment>
@@
 <segment>
 <pinref part="U1" gate="G$1" pin="TXD0"/>
-<wire x1="210.82" y1="114.3" x2="215.9" y2="114.3" width="0.1524" layer="91"/>
+<wire x1="210.82" y1="114.3" x2="238.76" y2="111.76" width="0.1524" layer="91"/>
 <pinref part="R1" gate="G$1" pin="1"/>
 </segment>
@@
 <net name="TX0" class="0">
 <segment>
-<wire x1="226.06" y1="114.3" x2="233.68" y2="114.3" width="0.1524" layer="91"/>
-<label x="228.6" y="114.3" size="1.778" layer="95"/>
+<wire x1="248.92" y1="111.76" x2="251.46" y2="111.76" width="0.1524" layer="91"/>
+<label x="251.46" y="111.76" size="1.778" layer="95"/>
 <pinref part="R1" gate="G$1" pin="2"/>
 </segment>
@@
 <segment>
 <pinref part="U1" gate="G$1" pin="SCK/CLK"/>
-<wire x1="210.82" y1="119.38" x2="215.9" y2="119.38" width="0.1524" layer="91"/>
-<wire x1="215.9" y1="119.38" x2="215.9" y2="121.92" width="0.1524" layer="91"/>
-<wire x1="215.9" y1="121.92" x2="228.6" y2="121.92" width="0.1524" layer="91"/>
-<wire x1="228.6" y1="121.92" x2="228.6" y2="119.38" width="0.1524" layer="91"/>
-<wire x1="228.6" y1="119.38" x2="233.68" y2="119.38" width="0.1524" layer="91"/>
+<wire x1="210.82" y1="119.38" x2="215.9" y2="116.84" width="0.1524" layer="91"/>
+<wire x1="215.9" y1="116.84" x2="233.68" y2="116.84" width="0.1524" layer="91"/>
 <label x="228.6" y="119.38" size="1.778" layer="95"/>
-<wire x1="215.9" y1="121.92" x2="215.9" y2="124.46" width="0.1524" layer="91"/>
-<wire x1="215.9" y1="124.46" x2="233.68" y2="124.46" width="0.1524" layer="91"/>
-<junction x="215.9" y="121.92"/>
-<label x="226.06" y="124.46" size="1.778" layer="95"/>
+<wire x1="215.9" y1="116.84" x2="215.9" y2="119.38" width="0.1524" layer="91"/>
+<wire x1="215.9" y1="119.38" x2="233.68" y2="119.38" width="0.1524" layer="91"/>
+<junction x="215.9" y="116.84"/>
+<label x="228.6" y="121.92" size="1.778" layer="95"/>
 </segment>
 <segment>
@@
 <segment>
 <pinref part="U1" gate="G$1" pin="IO35"/>
-<wire x1="210.82" y1="111.76" x2="233.68" y2="111.76" width="0.1524" layer="91"/>
+<wire x1="210.82" y1="111.76" x2="233.68" y2="109.22" width="0.1524" layer="91"/>
 <label x="213.36" y="111.76" size="1.778" layer="95"/>
 </segment>
@@
 <label x="287.02" y="99.06" size="1.778" layer="95"/>
 </segment>
+<segment>
+<pinref part="U1" gate="G$1" pin="SENSOR_VP"/>
+<wire x1="180.34" y1="139.7" x2="165.1" y2="139.7" width="0.1524" layer="91"/>
+<label x="165.1" y="139.7" size="1.778" layer="95"/>
+</segment>
 </net>
 <net name="MSGEQ_OUT" class="0">
@@
 <segment>
 <pinref part="U1" gate="G$1" pin="IO34"/>
-<wire x1="210.82" y1="109.22" x2="233.68" y2="109.22" width="0.1524" layer="91"/>
+<wire x1="210.82" y1="109.22" x2="233.68" y2="106.68" width="0.1524" layer="91"/>
 <label x="218.44" y="109.22" size="1.778" layer="95"/>
 </segment>
@@
 </segment>
 <segment>
-<pinref part="U1" gate="G$1" pin="IO22"/>
-<wire x1="180.34" y1="104.14" x2="165.1" y2="104.14" width="0.1524" layer="91"/>
-<label x="165.1" y="104.14" size="1.778" layer="95"/>
+<pinref part="U1" gate="G$1" pin="IO23"/>
+<wire x1="180.34" y1="101.6" x2="165.1" y2="101.6" width="0.1524" layer="91"/>
+<label x="165.1" y="101.6" size="1.778" layer="95"/>
 </segment>
 </net>
@@
 <segment>
 <pinref part="U1" gate="G$1" pin="SCS/CMD"/>
-<wire x1="210.82" y1="121.92" x2="213.36" y2="121.92" width="0.1524" layer="91"/>
-<wire x1="213.36" y1="121.92" x2="213.36" y2="127" width="0.1524" layer="91"/>
-<wire x1="213.36" y1="127" x2="233.68" y2="127" width="0.1524" layer="91"/>
-<label x="226.06" y="127" size="1.778" layer="95"/>
+<wire x1="210.82" y1="121.92" x2="218.44" y2="121.92" width="0.1524" layer="91"/>
+<label x="233.68" y="121.92" size="1.778" layer="95"/>
+<wire x1="218.44" y1="121.92" x2="233.68" y2="124.46" width="0.1524" layer="91"/>
 </segment>
 <segment>
@@
 </segment>
 <segment>
-<pinref part="U1" gate="G$1" pin="IO26"/>
-<wire x1="210.82" y1="99.06" x2="233.68" y2="99.06" width="0.1524" layer="91"/>
-<label x="226.06" y="99.06" size="1.778" layer="95"/>
+<pinref part="U1" gate="G$1" pin="SHD/SD2"/>
+<wire x1="210.82" y1="127" x2="220.98" y2="127" width="0.1524" layer="91"/>
+<label x="215.9" y="127" size="1.778" layer="95"/>
 </segment>
 </net>
@@
 </segment>
 <segment>
-<pinref part="U1" gate="G$1" pin="IO27"/>
-<wire x1="210.82" y1="101.6" x2="233.68" y2="101.6" width="0.1524" layer="91"/>
-<label x="226.06" y="101.6" size="1.778" layer="95"/>
+<pinref part="U1" gate="G$1" pin="SWP/SD3"/>
+<wire x1="210.82" y1="124.46" x2="218.44" y2="124.46" width="0.1524" layer="91"/>
+<label x="215.9" y="124.46" size="1.778" layer="95"/>
 </segment>
 </net>
@@
 <label x="104.14" y="91.44" size="1.778" layer="95"/>
 </segment>
+<segment>
+<pinref part="U1" gate="G$1" pin="IO12"/>
+<wire x1="180.34" y1="121.92" x2="165.1" y2="121.92" width="0.1524" layer="91"/>
+<label x="165.1" y="121.92" size="1.778" layer="95"/>
+</segment>
 </net>
 <net name="OLED_CS" class="0">
 <segment>
 <pinref part="U1" gate="G$1" pin="IO33"/>
-<wire x1="210.82" y1="106.68" x2="233.68" y2="106.68" width="0.1524" layer="91"/>
+<wire x1="210.82" y1="106.68" x2="233.68" y2="104.14" width="0.1524" layer="91"/>
 <label x="220.98" y="106.68" size="1.778" layer="95"/>
 </segment>
@@
 <segment>
 <pinref part="U1" gate="G$1" pin="IO32"/>
-<wire x1="210.82" y1="104.14" x2="233.68" y2="104.14" width="0.1524" layer="91"/>
-<label x="220.98" y="104.14" size="1.778" layer="95"/>
+<wire x1="210.82" y1="104.14" x2="233.68" y2="101.6" width="0.1524" layer="91"/>
+<label x="223.52" y="101.6" size="1.778" layer="95"/>
 </segment>
 <segment>
@@
 </net>
 <net name="ROTARY_BUTTON_IN" class="0">
-<segment>
-<pinref part="U1" gate="G$1" pin="SENSOR_VP"/>
-<wire x1="180.34" y1="139.7" x2="165.1" y2="139.7" width="0.1524" layer="91"/>
-<label x="154.94" y="139.7" size="1.778" layer="95"/>
-</segment>
 <segment>
 <pinref part="R16" gate="G$1" pin="2"/>
@@
 <label x="88.9" y="55.88" size="1.778" layer="95"/>
 </segment>
-</net>
-<net name="N$16" class="0">
-<segment>
-<pinref part="U1" gate="G$1" pin="IO23"/>
-<wire x1="180.34" y1="101.6" x2="165.1" y2="101.6" width="0.1524" layer="91"/>
-</segment>
-</net>
-<net name="VDD3V3_TEMP-OUT" class="0">
-<segment>
-<pinref part="U1" gate="G$1" pin="IO12"/>
-<wire x1="180.34" y1="121.92" x2="165.1" y2="121.92" width="0.1524" layer="91"/>
-<label x="165.1" y="121.92" size="1.778" layer="95"/>
-</segment>
-</net>
+<segment>
+<pinref part="U1" gate="G$1" pin="IO14"/>
+<wire x1="180.34" y1="116.84" x2="165.1" y2="116.84" width="0.1524" layer="91"/>
+<label x="154.94" y="116.84" size="1.778" layer="95"/>
+</segment>
+</net>

Commit message: omg
Connections:
- net LEDS8_3V3: now also U1.IO22; no longer U1.IO23
- net MSGEQ_RST: now also U1.IO27; no longer U1.SENSOR_VP
Other:
- moved on the sheet: C1, R1, R16
Changed lines of the file:
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@@
 <attribute name="VALUE" x="377.19" y="171.958" size="1.778" layer="96"/>
 </instance>
-<instance part="R1" gate="G$1" x="243.84" y="111.76" smashed="yes">
-<attribute name="NAME" x="237.49" y="110.7186" size="1.778" layer="95"/>
-<attribute name="VALUE" x="242.57" y="113.538" size="1.778" layer="96"/>
+<instance part="R1" gate="G$1" x="241.3" y="114.3" smashed="yes">
+<attribute name="NAME" x="234.95" y="113.2586" size="1.778" layer="95"/>
+<attribute name="VALUE" x="240.03" y="116.078" size="1.778" layer="96"/>
 </instance>
 <instance part="R10" gate="G$1" x="99.06" y="132.08" smashed="yes">
@@
 <attribute name="VALUE" x="115.062" y="189.23" size="1.778" layer="96"/>
 </instance>
-<instance part="C1" gate="G$1" x="106.68" y="30.48" smashed="yes" rot="R180">
-<attribute name="NAME" x="107.696" y="28.575" size="1.778" layer="95"/>
-<attribute name="VALUE" x="107.696" y="33.909" size="1.778" layer="96"/>
+<instance part="C1" gate="G$1" x="124.46" y="30.48" smashed="yes" rot="R180">
+<attribute name="NAME" x="125.476" y="28.575" size="1.778" layer="95"/>
+<attribute name="VALUE" x="125.476" y="33.909" size="1.778" layer="96"/>
 </instance>
 <instance part="C8" gate="G$1" x="76.2" y="30.48" smashed="yes" rot="R180">
@@
 <attribute name="VALUE" x="87.122" y="49.53" size="1.778" layer="96" rot="R90"/>
 </instance>
-<instance part="R16" gate="G$1" x="93.98" y="48.26" smashed="yes" rot="R90">
-<attribute name="NAME" x="92.4814" y="44.45" size="1.778" layer="95" rot="R90"/>
-<attribute name="VALUE" x="97.282" y="44.45" size="1.778" layer="96" rot="R90"/>
+<instance part="R16" gate="G$1" x="99.06" y="40.64" smashed="yes">
+<attribute name="NAME" x="95.25" y="42.1386" size="1.778" layer="95"/>
+<attribute name="VALUE" x="95.25" y="37.338" size="1.778" layer="96"/>
 </instance>
 <instance part="U5" gate="G$1" x="459.74" y="88.9" smashed="yes">
@@
 </segment>
 <segment>
-<wire x1="106.68" y1="35.56" x2="106.68" y2="63.5" width="0.1524" layer="91"/>
-<wire x1="76.2" y1="35.56" x2="63.5" y2="43.18" width="0.1524" layer="91"/>
-<wire x1="63.5" y1="43.18" x2="83.82" y2="63.5" width="0.1524" layer="91"/>
-<label x="116.84" y="55.88" size="1.778" layer="95"/>
-<wire x1="83.82" y1="63.5" x2="106.68" y2="63.5" width="0.1524" layer="91"/>
+<wire x1="124.46" y1="35.56" x2="124.46" y2="63.5" width="0.1524" layer="91"/>
+<wire x1="76.2" y1="35.56" x2="76.2" y2="43.18" width="0.1524" layer="91"/>
+<wire x1="76.2" y1="43.18" x2="76.2" y2="63.5" width="0.1524" layer="91"/>
+<label x="116.84" y="66.04" size="1.778" layer="95"/>
+<wire x1="76.2" y1="63.5" x2="124.46" y2="63.5" width="0.1524" layer="91"/>
 <pinref part="C1" gate="G$1" pin="2"/>
 <pinref part="C8" gate="G$1" pin="2"/>
 <pinref part="U$2" gate="G$1" pin="4"/>
 <wire x1="88.9" y1="35.56" x2="88.9" y2="43.18" width="0.1524" layer="91"/>
-<wire x1="88.9" y1="43.18" x2="63.5" y2="43.18" width="0.1524" layer="91"/>
-<junction x="63.5" y="43.18"/>
+<wire x1="88.9" y1="43.18" x2="76.2" y2="43.18" width="0.1524" layer="91"/>
+<junction x="76.2" y="43.18"/>
 </segment>
 <segment>
@@
 <segment>
 <pinref part="U1" gate="G$1" pin="RXD0"/>
-<wire x1="210.82" y1="116.84" x2="233.68" y2="114.3" width="0.1524" layer="91"/>
-<label x="228.6" y="116.84" size="1.778" layer="95"/>
+<wire x1="210.82" y1="116.84" x2="231.14" y2="116.84" width="0.1524" layer="91"/>
+<label x="218.44" y="116.84" size="1.778" layer="95"/>
 </segment>
 <segment>
@@
 <segment>
 <pinref part="U1" gate="G$1" pin="TXD0"/>
-<wire x1="210.82" y1="114.3" x2="238.76" y2="111.76" width="0.1524" layer="91"/>
+<wire x1="210.82" y1="114.3" x2="236.22" y2="114.3" width="0.1524" layer="91"/>
 <pinref part="R1" gate="G$1" pin="1"/>
 </segment>
@@
 <net name="TX0" class="0">
 <segment>
-<wire x1="248.92" y1="111.76" x2="251.46" y2="111.76" width="0.1524" layer="91"/>
-<label x="251.46" y="111.76" size="1.778" layer="95"/>
+<wire x1="246.38" y1="114.3" x2="251.46" y2="114.3" width="0.1524" layer="91"/>
+<label x="251.46" y="114.3" size="1.778" layer="95"/>
 <pinref part="R1" gate="G$1" pin="2"/>
 </segment>
@@
 <segment>
 <pinref part="U1" gate="G$1" pin="SCK/CLK"/>
-<wire x1="210.82" y1="119.38" x2="215.9" y2="116.84" width="0.1524" layer="91"/>
-<wire x1="215.9" y1="116.84" x2="233.68" y2="116.84" width="0.1524" layer="91"/>
-<label x="228.6" y="119.38" size="1.778" layer="95"/>
-<wire x1="215.9" y1="116.84" x2="215.9" y2="119.38" width="0.1524" layer="91"/>
-<wire x1="215.9" y1="119.38" x2="233.68" y2="119.38" width="0.1524" layer="91"/>
-<junction x="215.9" y="116.84"/>
-<label x="228.6" y="121.92" size="1.778" layer="95"/>
+<wire x1="210.82" y1="119.38" x2="248.92" y2="119.38" width="0.1524" layer="91"/>
+<wire x1="248.92" y1="119.38" x2="266.7" y2="119.38" width="0.1524" layer="91"/>
+<label x="254" y="119.38" size="1.778" layer="95"/>
+<wire x1="248.92" y1="119.38" x2="248.92" y2="129.54" width="0.1524" layer="91"/>
+<wire x1="248.92" y1="129.54" x2="266.7" y2="129.54" width="0.1524" layer="91"/>
+<junction x="248.92" y="119.38"/>
+<label x="254" y="129.54" size="1.778" layer="95"/>
 </segment>
 <segment>
@@
 <segment>
 <pinref part="U1" gate="G$1" pin="IO35"/>
-<wire x1="210.82" y1="111.76" x2="233.68" y2="109.22" width="0.1524" layer="91"/>
+<wire x1="210.82" y1="111.76" x2="233.68" y2="111.76" width="0.1524" layer="91"/>
 <label x="213.36" y="111.76" size="1.778" layer="95"/>
 </segment>
@@
 </segment>
 <segment>
-<pinref part="U1" gate="G$1" pin="SENSOR_VP"/>
-<wire x1="180.34" y1="139.7" x2="165.1" y2="139.7" width="0.1524" layer="91"/>
-<label x="165.1" y="139.7" size="1.778" layer="95"/>
+<pinref part="U1" gate="G$1" pin="IO27"/>
+<wire x1="210.82" y1="101.6" x2="233.68" y2="101.6" width="0.1524" layer="91"/>
+<label x="220.98" y="101.6" size="1.778" layer="95"/>
 </segment>
 </net>
@@
 <segment>
 <pinref part="U1" gate="G$1" pin="IO34"/>
-<wire x1="210.82" y1="109.22" x2="233.68" y2="106.68" width="0.1524" layer="91"/>
+<wire x1="210.82" y1="109.22" x2="233.68" y2="109.22" width="0.1524" layer="91"/>
 <label x="218.44" y="109.22" size="1.778" layer="95"/>
 </segment>
@@
 <pinref part="U1" gate="G$1" pin="IO4"/>
 <wire x1="180.34" y1="127" x2="165.1" y2="127" width="0.1524" layer="91"/>
-<label x="154.94" y="127" size="1.778" layer="95"/>
+<label x="162.56" y="127" size="1.778" layer="95"/>
 </segment>
 </net>
@@
 </segment>
 <segment>
-<pinref part="U1" gate="G$1" pin="IO23"/>
-<wire x1="180.34" y1="101.6" x2="165.1" y2="101.6" width="0.1524" layer="91"/>
-<label x="165.1" y="101.6" size="1.778" layer="95"/>
+<pinref part="U1" gate="G$1" pin="IO22"/>
+<wire x1="180.34" y1="104.14" x2="165.1" y2="104.14" width="0.1524" layer="91"/>
+<label x="165.1" y="104.14" size="1.778" layer="95"/>
 </segment>
 </net>
@@
 <segment>
 <pinref part="U1" gate="G$1" pin="SCS/CMD"/>
-<wire x1="210.82" y1="121.92" x2="218.44" y2="121.92" width="0.1524" layer="91"/>
-<label x="233.68" y="121.92" size="1.778" layer="95"/>
-<wire x1="218.44" y1="121.92" x2="233.68" y2="124.46" width="0.1524" layer="91"/>
+<label x="226.06" y="121.92" size="1.778" layer="95"/>
+<wire x1="210.82" y1="121.92" x2="231.14" y2="121.92" width="0.1524" layer="91"/>
 </segment>
 <segment>
@@
 <wire x1="96.52" y1="20.32" x2="96.52" y2="7.62" width="0.1524" layer="91"/>
 <label x="96.52" y="7.62" size="1.778" layer="95" rot="R90"/>
-<wire x1="96.52" y1="20.32" x2="106.68" y2="20.32" width="0.1524" layer="91"/>
-<wire x1="106.68" y1="20.32" x2="106.68" y2="27.94" width="0.1524" layer="91"/>
+<wire x1="96.52" y1="20.32" x2="124.46" y2="20.32" width="0.1524" layer="91"/>
+<wire x1="124.46" y1="20.32" x2="124.46" y2="27.94" width="0.1524" layer="91"/>
 <pinref part="U$2" gate="G$1" pin="2"/>
 <junction x="96.52" y="20.32"/>
@@
 <pinref part="U1" gate="G$1" pin="IO12"/>
 <wire x1="180.34" y1="121.92" x2="165.1" y2="121.92" width="0.1524" layer="91"/>
-<label x="165.1" y="121.92" size="1.778" layer="95"/>
+<label x="154.94" y="121.92" size="1.778" layer="95"/>
 </segment>
 </net>
@@
 <segment>
 <pinref part="U1" gate="G$1" pin="IO33"/>
-<wire x1="210.82" y1="106.68" x2="233.68" y2="104.14" width="0.1524" layer="91"/>
+<wire x1="210.82" y1="106.68" x2="233.68" y2="106.68" width="0.1524" layer="91"/>
 <label x="220.98" y="106.68" size="1.778" layer="95"/>
 </segment>
@@
 <segment>
 <pinref part="U1" gate="G$1" pin="IO32"/>
-<wire x1="210.82" y1="104.14" x2="233.68" y2="101.6" width="0.1524" layer="91"/>
-<label x="223.52" y="101.6" size="1.778" layer="95"/>
+<wire x1="210.82" y1="104.14" x2="236.22" y2="104.14" width="0.1524" layer="91"/>
+<label x="223.52" y="104.14" size="1.778" layer="95"/>
 </segment>
 <segment>
@@
 <pinref part="U$2" gate="G$1" pin="5"/>
 <pinref part="R16" gate="G$1" pin="1"/>
-<wire x1="93.98" y1="35.56" x2="93.98" y2="43.18" width="0.1524" layer="91"/>
+<wire x1="93.98" y1="35.56" x2="93.98" y2="40.64" width="0.1524" layer="91"/>
 </segment>
 </net>
@@
 <segment>
 <pinref part="R16" gate="G$1" pin="2"/>
-<wire x1="93.98" y1="53.34" x2="88.9" y2="53.34" width="0.1524" layer="91"/>
-<wire x1="88.9" y1="53.34" x2="88.9" y2="45.72" width="0.1524" layer="91"/>
+<wire x1="104.14" y1="40.64" x2="104.14" y2="48.26" width="0.1524" layer="91"/>
+<wire x1="104.14" y1="48.26" x2="83.82" y2="48.26" width="0.1524" layer="91"/>
 <pinref part="R11" gate="G$1" pin="1"/>
-<wire x1="88.9" y1="45.72" x2="83.82" y2="45.72" width="0.1524" layer="91"/>
-<wire x1="83.82" y1="45.72" x2="83.82" y2="48.26" width="0.1524" layer="91"/>
-<wire x1="88.9" y1="53.34" x2="88.9" y2="55.88" width="0.1524" layer="91"/>
-<wire x1="88.9" y1="55.88" x2="96.52" y2="55.88" width="0.1524" layer="91"/>
-<junction x="88.9" y="53.34"/>
-<label x="88.9" y="55.88" size="1.778" layer="95"/>
-</segment>
-<segment>
+<wire x1="104.14" y1="48.26" x2="116.84" y2="48.26" width="0.1524" layer="91"/>
+<junction x="104.14" y="48.26"/>
+<label x="96.52" y="50.8" size="1.778" layer="95"/>
+</segment>
+<segment>

Commit message: Another day closer to death...
Connections:
- net GAIN: now also U1.IO26
Changed lines of the file:
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@@
 <label x="441.96" y="121.92" size="1.778" layer="95"/>
+</segment>
+<segment>
+<pinref part="U1" gate="G$1" pin="IO26"/>
+<wire x1="210.82" y1="99.06" x2="233.68" y2="99.06" width="0.1524" layer="91"/>
+<label x="223.52" y="99.06" size="1.778" layer="95"/>
 </segment>
 </net>
