File: Lamp Logic Board/Lamp Logic Board_3.brd (EAGLE design)
At the start: 41.5 x 84.8 mm, 45 parts, among them U1 ESP32-WROVER-IB, U2 SN74HCT245DWR, U4 LM50, U5 SPIOLED_STANDOFF, U6 MSGEQ7DIL

Commit message: Another day closer to death...
Parts:
- removed PAD5V, PAD5V1, PADGND, PADGND1: (no value), wirepad:SMD2,54-5,08
- moved R10 43.3 mm to (-30.6, 69.6)
- moved S1 37.4 mm to (-28.0, 61.7)
- moved R12 29.3 mm to (-16.7, 60.6)
- moved MICROSD_CONN 26.5 mm to (27.9, 27.7)
- moved U$3 25.2 mm to (29.4, 39.5), turned to 270 degrees
- moved R14 23.8 mm to (-4.32, 41.3), turned to 270 degrees
- moved R13 23.4 mm to (-4.25, 35.4)
- moved S2 23.2 mm to (-12.4, 38.3)
- moved R1 19.6 mm to (9.22, 25.1), turned to 270 degrees
- moved U2 13.7 mm to (30.2, 48.1)
- moved C9 12.6 mm to (10.9, 62.7), turned to 90 degrees
- moved R2 11.9 mm to (12.2, 15.3)
- moved R3 11.7 mm to (15.2, 15.3)
- moved R4 11.5 mm to (18.2, 15.3)
- moved R5 11.4 mm to (21.1, 15.3)
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Connections:
- new net N$30: U1.37
- new net N$38: U1.20
- new net N$39: U1.19
- new net N$40: U1.18
- new net N$41: U1.17
- new net N$42: U1.22
- new net N$43: U1.21
- net CS: no longer U1.19
- net GAIN: no longer U1.11
- net GND: no longer PADGND.1, PADGND1.1
- net IO0: no longer U1.25
- net LEDS1_3V3: now also U1.33; no longer U1.23
- net LEDS2_3V3: now also U1.31; no longer U1.24
- net LEDS3_3V3: now also U1.30; no longer U1.26
- net LEDS4_3V3: now also U1.23; no longer U1.29
- net LEDS5_3V3: now also U1.24; no longer U1.30
- net LEDS6_3V3: now also U1.25; no longer U1.31
- net LEDS7_3V3: now also U1.26; no longer U1.33
- net LEDS8_3V3: now also U1.29; no longer U1.36
- net LEDSDIAG_3V3: no longer U1.16
- net MISO: now also U1.14; no longer U1.21
- net MOSI: now also U1.16; no longer U1.22
- net MSGEQ_OUT: now also U1.4; no longer U1.6
- net MSGEQ_RST: now also U1.9; no longer U1.12
- net MSGEQ_STROBE: now also U1.8; no longer U1.7
- net OLED_CS: no longer U1.9
- net OLED_DC: no longer U1.8
- net OUTA: now also U1.10, U1.7; no longer U1.17
- net OUTB: now also U1.12; no longer U1.18
- net ROTARY_BUTTON_IN: now also U1.11; no longer U1.13
- net SCK: now also U1.13; no longer U1.20
- net SD_CS: now also U1.36; no longer U1.10
- net VDD3V3_TEMP_OUT: now also U1.6; no longer U1.14
- net VDD5V: no longer PAD5V.1, PAD5V1.1
Routing:
- net VDD5V: track 236.2 -> 99.8 mm, vias 4 -> 2
- net GND: track 97.0 -> 3.57 mm, vias 0 -> 2
- net IO0: track 71.9 -> 0.00 mm, vias 2 -> 0
- net LEDS8_3V3: track 52.7 -> 18.0 mm, vias 2 -> 0
- net LEDS7_3V3: track 48.3 -> 13.8 mm, vias 2 -> 0
- net LEDS4_3V3: track 42.8 -> 8.91 mm, vias 2 -> 0
- net LEDS5_3V3: track 44.1 -> 10.3 mm, vias 2 -> 0
- net LEDS6_3V3: track 45.4 -> 12.0 mm, vias 2 -> 0
- net N$15: track 10.1 -> 42.6 mm, vias 0 -> 2
- net N$14: track 10.0 -> 40.2 mm, vias 0 -> 2
- net N$13: track 7.74 -> 37.8 mm, vias 0 -> 2
- net N$12: track 6.31 -> 35.4 mm, vias 0 -> 2
- net N$2: track 49.7 -> 78.1 mm
- net N$11: track 5.20 -> 33.0 mm, vias 0 -> 2
- net N$10: track 4.61 -> 31.9 mm, vias 0 -> 2
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Other:
- board size 41.5 x 84.8 mm -> 37.2 x 81 mm

Commit message: still getting stuck on file 99
Parts:
- removed LED1: WS2812B5050, WS2812B:WS2812B
- removed U$1: XT60, XT60:XT60
- removed U$5: 2X4PINHEAD, 2X4PINHEAD:2X4PINHEAD
- added 5V_POWER_INPUT: XT60-M, XT60-M:AMASS_XT60-M
- added SERIAL/SPI_HEADER: 2X6PINHEAD, 2X4PINHEAD:2X6PINHEAD
- moved R10 42.5 mm to (5.35, 46.9), turned to 180 degrees
- moved S1 39.6 mm to (6.83, 42.9), turned to 0 degrees
- moved R12 29.5 mm to (9.50, 47.1), turned to 270 degrees
- moved R15 0.06 mm to (9.97, 8.03)
- renumbered MICROSD_CONN to SD_CARD_READER, MIC_CONN to MIC_HEADER, U$2 to ROTARY_ENCODER, U$3 to SD_CARD_FILTER, U$4 to 3X8_24_PIN_LED_OUTPUT, U2 to LOGIC_LEVEL_SHIFTER, U3 to 5V_TO_3V3_REGULATOR, U4 to TEMP_SENSOR, U5 to OLED_HEADER, U6 to MSGEQ7
Connections:
- net OUTB renamed ROTARY_OUT_B
- net ROTARY_BUTTON_IN renamed ROTARY_BUTTON_OUT
- net VDD3V3_TEMP_OUT renamed TEMP_OUT
- removed net CS: U$5.CS
- removed net LEDSDIAG_3V3: LED1.4-DIN
- removed net N$2: R1.1, U1.35
- removed net N$30: U1.37
- removed net N$38: U1.20
- removed net N$39: U1.19
- removed net N$40: U1.18
- removed net N$41: U1.17
- removed net N$42: U1.22
- removed net N$43: U1.21
- removed net OUTA: C8.1, ROTARY_ENCODER.1, U1.10, U1.7
- new net HEADER_CS: R1.1, SERIAL/SPI_HEADER.CS, U1.35
- new net ROTARY_OUT_A: C8.1, ROTARY_ENCODER.1, U1.10
- net EN: now also SERIAL/SPI_HEADER.DTR
- net GND: now also 5V_POWER_INPUT.1, SERIAL/SPI_HEADER.GND; no longer LED1.3-GND, U$1.-, U$5.GND
- net LEDS6_3V3: now also SERIAL/SPI_HEADER.RTS
- net MISO: now also SERIAL/SPI_HEADER.MISO; no longer U$5.MISO
- net MOSI: now also SERIAL/SPI_HEADER.MOSI; no longer U$5.MOSI
- net OLED_CS: now also U1.7
- net OLED_DC: now also U1.37
- net RX0: now also SERIAL/SPI_HEADER.RX0; no longer U$5.RX0
- net SCK: now also SERIAL/SPI_HEADER.SCK; no longer U$5.SCK
- net TX0: now also SERIAL/SPI_HEADER.TX0; no longer U$5.TX0
- net VDD3V3: now also SERIAL/SPI_HEADER.VCC; no longer U$5.VDD
- net VDD5V: now also 5V_POWER_INPUT.2; no longer LED1.1-VDD, U$1.+
Routing:
- net VDD5V: track 99.8 -> 204.8 mm, vias 2 -> 3
- net GND: track 3.57 -> 99.0 mm, vias 2 -> 6
- net HEADER_CS: track 0.00 -> 86.9 mm, vias 0 -> 2
- net N$2: track 78.1 -> 0.00 mm, vias 2 -> 0
- net EN: track 0.00 -> 67.9 mm, vias 0 -> 2
- net ROTARY_OUT_A: track 0.00 -> 42.3 mm, vias 0 -> 1
- net CS: track 37.4 -> 0.00 mm
- net OUTA: track 35.0 -> 0.00 mm
- net OLED_DC: track 28.2 -> 53.2 mm, vias 0 -> 3
- net OLED_CS: track 26.5 -> 35.2 mm, vias 0 -> 1
- net ROTARY_BUTTON_OUT: track 42.8 -> 48.6 mm, vias 1 -> 2
- net N$9: track 0.00 -> 4.05 mm
- net N$15: track 42.6 -> 46.5 mm
- net N$14: track 40.2 -> 44.1 mm
- net N$12: track 35.4 -> 39.3 mm
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
Commit message: and the rest
Parts:
- removed TEMP_SENSOR: LM50, linear:SOT23
- added C11, C12, C5: 100nF, resistor:C0402
- C9: value 0.01uF -> 1uF
- R12, R14: value (none) -> 12k
- moved S2 42.6 mm to (28.4, 26.2), flipped to the bottom, turned to 270 degrees
- moved C9 24.7 mm to (35.2, 58.5), turned to 180 degrees
- moved R13 24.4 mm to (10.2, 55.0), turned to 0 degrees
- moved R14 20.2 mm to (8.11, 57.2), turned to 0 degrees
- moved SD_CARD_FILTER 1.55 mm to (28.0, 38.8), turned to 0 degrees
- moved R10 1.12 mm to (4.30, 47.3)
- moved C3 0.89 mm to (21.0, 52.1), turned to 180 degrees
- moved C6 0.65 mm to (20.9, 47.8)
- moved S1 0.64 mm to (6.33, 43.3)
- moved R16 0.50 mm to (4.75, 25.1)
- moved R12 0.44 mm to (9.10, 47.3), turned to 180 degrees
- moved R1 0.35 mm to (9.57, 25.1)
- moved C2 0.30 mm to (9.22, 78.2)
- moved R15 0.08 mm to (9.90, 8.05)
Connections:
- removed net IO0: R13.1, R14.2
- removed net TEMP_OUT: TEMP_SENSOR.2, U1.6
- new net BEST_BUTTON: C11.1, R13.1, R14.2, U1.12
- net GND: now also C11.2, C12.1, C5.2; no longer TEMP_SENSOR.3
- net OLED_CS: now also U1.10; no longer U1.7
- net ROTARY_BUTTON_OUT: now also C12.2, U1.7; no longer U1.11
- net ROTARY_OUT_A: now also U1.6; no longer U1.10
- net ROTARY_OUT_B: now also U1.11; no longer U1.12
- net VDD3V3: no longer C9.1, TEMP_SENSOR.1
- net VDD5V: now also C5.1, C9.1
Routing:
- net N$7: track 0.00 -> 50.6 mm, vias 0 -> 3
- net LEDS6_3V3: track 12.3 -> 37.3 mm
- net GND: track 99.0 -> 121.0 mm, vias 6 -> 5
- net BEST_BUTTON: track 0.00 -> 18.0 mm, vias 0 -> 2
- net TEMP_OUT: track 14.9 -> 0.00 mm
- net HEADER_CS: track 86.9 -> 77.3 mm
- net MSGEQ_STROBE: track 20.0 -> 12.5 mm, vias 3 -> 1
- net ROTARY_BUTTON_OUT: track 48.6 -> 55.9 mm
- net ROTARY_OUT_A: track 42.3 -> 47.1 mm
- net MISO: track 63.8 -> 59.2 mm
- net MOSI: track 60.9 -> 56.3 mm
- net SD_CS: track 46.5 -> 42.5 mm
- net N$15: track 46.5 -> 42.6 mm
- net VDD5V: track 204.8 -> 208.8 mm
- net N$14: track 44.1 -> 40.2 mm
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
Commit message: everything but those two pesky caps
Parts:
- removed S2: (no value), SparkFun-Switches:TACTILE_SWITCH_SMD_6.0X3.5MM
- added S3: MOMENTARY-SWITCH-SPST-SMD-12MM, SparkFun-Switches:TACTILE_SWITCH_SMD_12MM
Connections:
- net GND: now also S3.3; no longer S2.2
- net N$7: now also S3.1; no longer S2.1
Routing:
- net HEADER_CS: track 77.3 -> 68.2 mm
- net N$12: track 41.2 -> 38.2 mm
- net N$11: track 38.8 -> 35.9 mm
- net N$15: track 42.6 -> 45.3 mm
- net N$14: track 40.2 -> 42.9 mm
- net N$13: track 38.3 -> 40.5 mm
- net EN: track 70.0 -> 67.8 mm
- net RX0: track 67.3 -> 65.3 mm
- net VDD5V: track 208.8 -> 210.7 mm
- net N$10: track 36.5 -> 34.7 mm
- net N$7: track 50.6 -> 49.2 mm
- net MISO: track 59.2 -> 60.6 mm, vias 3 -> 2
- net SD_CS: track 42.5 -> 43.3 mm
- net N$6: track 34.7 -> 34.0 mm
- net MOSI: track 56.3 -> 56.9 mm
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